File: uaeficopiedtovfr.kicad_pcb (KiCad board)
At the start: 2 copper layers, 160 x 75.1 mm, 66 parts, among them J1 DTF13-12PB, J4 DTF13-12PB, J9 USB_C_Receptacle_USB2.0, M1 Module-power_12and5V-0.2, M2 Module-knock-0.2, M3 Module-vr-discrete-0.4, M4 Module-vr-max9924-0.1, M5 Module-wbo-0.5, M6 Module:mega-mcu100/0.2, M7 Module-wbo-0.5, P3 Pad, P4 Pad, Q1 ISL9V3040D3S, Q10 ZXMS6005SGTA, Q11 AO3400A, Q12 AO3400A, Q13 ZXMS6005SGTA, Q14 ZXMS6005SGTA, Q15 ZXMS6005SGTA, Q16 ZXMS6005SGTA, Q2 ISL9V3040D3S, Q3 ISL9V3040D3S, Q4 ISL9V3040D3S, Q7 ZXMS6005SGTA, Q8 ZXMS6005SGTA, Q9 ZXMS6005SGTA, U2 JDY-33

Commit message: Update uaeficopiedtovfr.kicad_pcb
Parts:
- removed REF**: trollfaceVFR, Customparts:trollfaceVFR
- moved M5 9.45 mm to (97.7, 91.5), turned to -90 degrees
- moved M7 4.80 mm to (81.1, 95.9), turned to -90 degrees
Connections:
- J1 pad 1: +12V_RAW -> /WBO2_Heater
- J1 pad 10: /WBO2_Vm -> /WBO2_Un
- J1 pad 12: /WBO2_Un -> /WBO2_Vm
- J1 pad 3: /WBO2_Heater -> +12V_RAW
Routing:
- net /WBO2_Un: track 12.3 -> 37.4 mm
- net +5VA: track 345.8 -> 324.0 mm
- net /WBO_Rtrim: track 6.30 -> 28.1 mm
- net /WBO2_Rtrim: track 14.1 -> 34.7 mm
- net /WBO_Vm: track 13.2 -> 31.9 mm
- net /WBO_Ip: track 11.1 -> 29.3 mm
- net /WBO_Un: track 10.4 -> 28.4 mm
- net /WBO_Heater: track 10.8 -> 27.6 mm
- net /WBO2_Ip: track 16.8 -> 30.3 mm
- net /CAN-: track 150.7 -> 141.4 mm
- net /WBO2_Heater: track 17.6 -> 24.4 mm
- net /CAN+: track 149.8 -> 143.9 mm
- net /WBO2_Vm: track 21.2 -> 24.7 mm
- net +12V_RAW: track 249.0 -> 252.3 mm
- net GND: vias 47 -> 45
