File: uaeficopiedtovfr.kicad_sch (KiCad schematic)
At the start: 36 parts, among them J1 USB_B_Mini, J1 USB_C_Receptacle_USB2.0, J17 Conn_01x06, J4 1-776087-1, J5 Conn_01x05_Male, M1 Module-power_12and5V-0.2, M3 Module-knock-0.2, M3 Module-vr-discrete-0.4, M4 Module-vr-max9924-0.1, M5 Module-wbo-0.5, M6 Module:mega-mcu100/0.2, M7 Module-wbo-0.5, M8 Module-sd-0.1, P1 Pad, P2 Pad, P3 Pad, P4 Pad, U4 JDY-33

Commit message: Routed aux2 and button3 to rear connector
Routed aux2 and button3 to rear connector
Parts:
- removed M8: Module-sd-0.1, hellen-one-sd-0.1:sd, symbol hellen-one-sd:Module-sd-0.1
Connections:
- net GND: no longer J4.10, J4.11
- net IN_AUX2: now also J4.11
- net IN_BUTTON3: now also J4.10
- net PG_5VP: no longer M6.N12 (SPI3_MOSI_(PC12))
Changed lines of the file:
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@@
   (junction (at 334.01 344.17) (diameter 0) (color 0 0 0 0)
   )
-  (junction (at 429.26 135.89) (diameter 0) (color 0 0 0 0)
-  )
   (junction (at 20.32 72.39) (diameter 0) (color 0 0 0 0)
   )
   (junction (at 346.71 166.37) (diameter 0) (color 0 0 0 0)
   )
-  (junction (at 429.26 138.43) (diameter 0) (color 0 0 0 0)
-  )
   (junction (at 156.21 99.06) (diameter 0) (color 0 0 0 0)
   )
@@
     (stroke (width 0) (type default))
   )
-  (wire (pts (xy 429.26 138.43) (xy 429.26 135.89))
-    (stroke (width 0) (type default))
-  )
   (bus (pts (xy 208.28 135.89) (xy 208.28 138.43))
     (stroke (width 0) (type default) (color 255 153 0 1))
@@
     (stroke (width 0) (type default))
   )
-  (wire (pts (xy 427.99 125.73) (xy 430.53 125.73))
-    (stroke (width 0) (type default))
-  )
   (wire (pts (xy 256.54 186.69) (xy 256.54 168.91))
     (stroke (width 0) (type default))
@@
     (stroke (width 0) (type default))
   )
-  (wire (pts (xy 430.53 125.73) (xy 430.53 123.19))
-    (stroke (width 0) (type default))
-  )
-  (wire (pts (xy 341.63 125.73) (xy 384.81 125.73))
-    (stroke (width 0) (type default))
-  )
   (wire (pts (xy 260.35 270.51) (xy 273.05 270.51))
     (stroke (width 0) (type default))
@@
     (stroke (width 0) (type default))
   )
-  (wire (pts (xy 429.26 133.35) (xy 427.99 133.35))
-    (stroke (width 0) (type default))
-  )
   (wire (pts (xy 147.32 106.68) (xy 147.32 109.22))
     (stroke (width 0) (type default))
   )
-  (wire (pts (xy 375.92 133.35) (xy 384.81 133.35))
-    (stroke (width 0) (type default))
-  )
   (wire (pts (xy 265.43 104.14) (xy 265.43 115.57))
     (stroke (width 0) (type default))
@@
     (stroke (width 0) (type default))
   )
-  (wire (pts (xy 427.99 135.89) (xy 429.26 135.89))
-    (stroke (width 0) (type default))
-  )
   (wire (pts (xy 358.14 95.25) (xy 313.69 95.25))
     (stroke (width 0) (type default))
@@
     (stroke (width 0) (type default))
   )
-  (wire (pts (xy 429.26 135.89) (xy 429.26 133.35))
-    (stroke (width 0) (type default))
-  )
   (bus (pts (xy 191.77 -19.05) (xy 191.77 -16.51))
     (stroke (width 0) (type default))
@@
     (stroke (width 0) (type default) (color 255 0 255 1))
   )
+  (wire (pts (xy 228.6 247.65) (xy 228.6 250.19))
+    (stroke (width 0) (type default))
+  )
   (wire (pts (xy 237.49 234.95) (xy 237.49 288.29))
     (stroke (width 0) (type default))
@@
     (stroke (width 0) (type default))
   )
-  (wire (pts (xy 341.63 128.27) (xy 384.81 128.27))
-    (stroke (width 0) (type default))
-  )
   (wire (pts (xy 341.63 184.15) (xy 350.52 184.15))
     (stroke (width 0) (type solid))
@@
     (stroke (width 0) (type default) (color 194 194 0 1))
   )
-  (wire (pts (xy 427.99 138.43) (xy 429.26 138.43))
-    (stroke (width 0) (type default))
-  )
   (wire (pts (xy 246.38 186.69) (xy 256.54 186.69))
     (stroke (width 0) (type default))
@@
     (stroke (width 0) (type default))
   )
-  (wire (pts (xy 228.6 250.19) (xy 218.44 250.19))
+  (wire (pts (xy 218.44 250.19) (xy 228.6 250.19))
     (stroke (width 0) (type default))
   )
@@
     (stroke (width 0) (type solid))
   )
-  (wire (pts (xy 384.81 130.81) (xy 341.63 130.81))
-    (stroke (width 0) (type default))
-  )
   (wire (pts (xy 124.46 119.38) (xy 111.76 119.38))
     (stroke (width 0) (type default))
@@
     (effects (font (size 1.27 1.27)) (justify right bottom))
   )
+  (label "IN_BUTTON3" (at 25.4 222.25 180) (fields_autoplaced)
+    (effects (font (size 1.27 1.27)) (justify right bottom))
+  )
   (label "IN_KNOCK_RAW" (at 129.54 186.69 0) (fields_autoplaced)
     (effects (font (size 1.27 1.27)) (justify left bottom))
@@
     (effects (font (size 1.27 1.27)) (justify left bottom))
   )
-  (label "VR2" (at 227.33 250.19 180) (fields_autoplaced)
+  (label "VR2" (at 228.6 247.65 180) (fields_autoplaced)
     (effects (font (size 1.27 1.27)) (justify right bottom))
   )
@@
     (effects (font (size 1.27 1.27)) (justify left bottom))
   )
-  (label "PGND" (at 25.4 224.79 180) (fields_autoplaced)
+  (label "IN_AUX2" (at 25.4 224.79 180) (fields_autoplaced)
     (effects (font (size 1.27 1.27)) (justify right bottom))
   )
@@
     (effects (font (size 1.27 1.27)) (justify right bottom))
   )
-  (label "PGND" (at 25.4 222.25 180) (fields_autoplaced)
-    (effects (font (size 1.27 1.27)) (justify right bottom))
-  )
   (label "IN_MAP" (at 133.35 199.39 0) (fields_autoplaced)
     (effects (font (size 1.27 1.27)) (justify left bottom))
@@
     )
   )
-  (symbol (lib_id "power:GND") (at 429.26 138.43 0) (unit 1)
-    (in_bom yes) (on_board yes) (dnp no) (fields_autoplaced)
-    (property "Reference" "#PWR09" (at 429.26 144.78 0)
-      (effects (font (size 1.27 1.27)) hide)
-    )
-    (property "Value" "GND" (at 429.26 143.51 0)
-      (effects (font (size 1.27 1.27)))
-    )
-    (property "Footprint" "" (at 429.26 138.43 0)
-      (effects (font (size 1.27 1.27)) hide)
-    )
-    (property "Datasheet" "" (at 429.26 138.43 0)
-      (effects (font (size 1.27 1.27)) hide)
-    )
-    (pin "1")
-    (instances
-      (project "uaeficopiedtovfr"
-        (path "/90b72e19-92bc-40db-bd4d-f17fb5de93ea"
-          (reference "#PWR09") (unit 1)
-        )
-      )
-    )
-  )
   (symbol (lib_id "power:GND") (at 367.03 74.93 0) (mirror y) (unit 1)
     (in_bom yes) (on_board yes) (dnp no)
@@
     )
   )
-  (symbol (lib_id "hellen-one-sd:Module-sd-0.1") (at 389.89 120.65 0) (unit 1)
-    (in_bom yes) (on_board yes) (dnp no) (fields_autoplaced)
-    (property "Reference" "M8" (at 406.4 116.84 0)
-      (effects (font (size 1.27 1.27)))
-    )
-    (property "Value" "Module-sd-0.1" (at 406.4 119.38 0)
-      (effects (font (size 1.27 1.27)))
-    )
-    (property "Footprint" "hellen-one-sd-0.1:sd" (at 389.89 120.65 0)
-      (effects (font (size 1.27 1.27)) hide)
-    )
-    (property "Datasheet" "" (at 389.89 120.65 0)
-      (effects (font (size 1.27 1.27)) hide)
-    )
-    (pin "G")
-    (pin "V1")
-    (pin "V2")
-    (pin "V3")
-    (pin "V4")
-    (pin "V5")
-    (pin "V6")
-    (pin "V7")
-    (instances
-      (project "uaeficopiedtovfr"
-        (path "/90b72e19-92bc-40db-bd4d-f17fb5de93ea"
-          (reference "M8") (unit 1)
-        )
-      )
-    )
-  )
   (symbol (lib_id "customparts:VFR_PCB") (at 39.37 104.14 90) (unit 1)
     (in_bom yes) (on_board yes) (dnp no) (fields_autoplaced)
@@
         )
       )
-    )
-  )
-  (symbol (lib_id "power:+3.3VA") (at 430.53 123.19 0) (unit 1)
-    (in_bom yes) (on_board yes) (dnp no)
-    (property "Reference" "#PWR075" (at 430.53 127 0)
-      (effects (font (size 1.27 1.27)) hide)
-    )
-    (property "Value" "+3.3VA" (at 426.72 119.38 0)
-      (effects (font (size 1.27 1.27)) (justify left))
-    )
-    (property "Footprint" "" (at 430.53 123.19 0)
-      (effects (font (size 1.27 1.27)) hide)
-    )
-    (property "Datasheet" "" (at 430.53 123.19 0)
-      (effects (font (size 1.27 1.27)) hide)
-    )
-    (pin "1")
-    (instances
-      (project "alphax_8ch"
-        (path "/63d2dd9f-d5ff-4811-a88d-0ba932475460/5e6758cb-9f53-4408-bcb6-fb57a3a22748"
-          (reference "#PWR075") (unit 1)
-        )
-      )
-      (project "uaeficopiedtovfr"
-        (path "/90b72e19-92bc-40db-bd4d-f17fb5de93ea"
-          (reference "#PWR057") (unit 1)
-        )
-      )
-      (project "uaefi"
-        (path "/ac264c30-3e9a-4be2-b97a-9949b68bd497"
-          (reference "#PWR051") (unit 1)
-        )
-      )
